Commit message: updated xml tags

File: tesseract_support/urdf/xarm7.urdf (robot description, URDF)
Before this commit: robot UF_ROBOT, 10 links, 9 joints
Links:
- removed link link_base
- removed link link_eef
- added link base
- added link base_link, mass 0.88556; collision mesh filename=/home/febert/code/xarm_ros_workspace/src/xarm_ros/xarm_desc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; visual mesh filename=/home/febert/code/xarm_ros_workspace/src/xarm_ros/xarm_desc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
- added link tool0
Joints:
- added joint base_link-base: type fixed, parent base_link, child base, origin xyz=0 0 0 rpy=0 0 0
- joint joint1: parent link_base -> base_link
- joint joint_eef: child link_eef -> tool0
- joint world_joint: child link_base -> base_link
