Commit message: added easo 1.0 files

File: tesseract_support/urdf/easo1.0_base_macro.xacro (robot description, xacro)
@@ -12,11 +12,50 @@
       <material name="light_gray"/>
     </visual>
+    <collision><geometry><mesh filename="package://tesseract_support/meshes/easo1.0/convex_decomposition/robot_base_decomposition_meshes/untitled_home_febert_Desktop_arm_base000_home_febert_Desktop_arm_base004.stl" /></geometry></collision>
+    <collision><geometry><mesh filename="package://tesseract_support/meshes/easo1.0/convex_decomposition/robot_base_decomposition_meshes/untitled_home_febert_Desktop_arm_base000_home_febert_Desktop_arm_base046.stl" /></geometry></collision>
+    <collision><geometry><mesh filename="package://tesseract_support/meshes/easo1.0/convex_decomposition/robot_base_decomposition_meshes/untitled_home_febert_Desktop_arm_base000_home_febert_Desktop_arm_base045.stl" /></geometry></collision>
+    <collision><geometry><mesh filename="package://tesseract_support/meshes/easo1.0/convex_decomposition/robot_base_decomposition_meshes/untitled_home_febert_Desktop_arm_base000_home_febert_Desktop_arm_base021.stl" /></geometry></collision>
+    <collision><geometry><mesh filename="package://tesseract_support/meshes/easo1.0/convex_decomposition/robot_base_decomposition_meshes/untitled_home_febert_Desktop_arm_base000_home_febert_Desktop_arm_base057.stl" /></geometry></collision>
+    <collision><geometry><mesh filename="package://tesseract_support/meshes/easo1.0/convex_decomposition/robot_base_decomposition_meshes/untitled_home_febert_Desktop_arm_base000_home_febert_Desktop_arm_base001.stl" /></geometry></collision>
+    <collision><geometry><mesh filename="package://tesseract_support/meshes/easo1.0/convex_decomposition/robot_base_decomposition_meshes/untitled_home_febert_Desktop_arm_base000_home_febert_Desktop_arm_base039.stl" /></geometry></collision>
+    <collision><geometry><mesh filename="package://tesseract_support/meshes/easo1.0/convex_decomposition/robot_base_decomposition_meshes/untitled_home_febert_Desktop_arm_base000_home_febert_Desktop_arm_base014.stl" /></geometry></collision>
+    <collision><geometry><mesh filename="package://tesseract_support/meshes/easo1.0/convex_decomposition/robot_base_decomposition_meshes/untitled_home_febert_Desktop_arm_base000_home_febert_Desktop_arm_base031.stl" /></geometry></collision>
+    <collision><geometry><mesh filename="package://tesseract_support/meshes/easo1.0/convex_decomposition/robot_base_decomposition_meshes/untitled_home_febert_Desktop_arm_base000_home_febert_Desktop_arm_base061.stl" /></geometry></collision>
+    <collision><geometry><mesh filename="package://tesseract_support/meshes/easo1.0/convex_decomposition/robot_base_decomposition_meshes/untitled_home_febert_Desktop_arm_base000_home_febert_Desktop_arm_base038.stl" /></geometry></collision>
+    <collision><geometry><mesh filename="package://tesseract_support/meshes/easo1.0/convex_decomposition/robot_base_decomposition_meshes/untitled_home_febert_Desktop_arm_base000_home_febert_Desktop_arm_base030.stl" /></geometry></collision>
+    <collision><geometry><mesh filename="package://tesseract_support/meshes/easo1.0/convex_decomposition/robot_base_decomposition_meshes/untitled_home_febert_Desktop_arm_base000_home_febert_Desktop_arm_base017.stl" /></geometry></collision>
+    <collision><geometry><mesh filename="package://tesseract_support/meshes/easo1.0/convex_decomposition/robot_base_decomposition_meshes/untitled_home_febert_Desktop_arm_base000_home_febert_Desktop_arm_base024.stl" /></geometry></collision>
+    <collision><geometry><mesh filename="package://tesseract_support/meshes/easo1.0/convex_decomposition/robot_base_decomposition_meshes/untitled_home_febert_Desktop_arm_base000_home_febert_Desktop_arm_base035.stl" /></geometry></collision>
+    <collision><geometry><mesh filename="package://tesseract_support/meshes/easo1.0/convex_decomposition/robot_base_decomposition_meshes/untitled_home_febert_Desktop_arm_base000_home_febert_Desktop_arm_base058.stl" /></geometry></collision>
+    <collision><geometry><mesh filename="package://tesseract_support/meshes/easo1.0/convex_decomposition/robot_base_decomposition_meshes/untitled_home_febert_Desktop_arm_base000_home_febert_Desktop_arm_base027.stl" /></geometry></collision>
+    <collision><geometry><mesh filename="package://tesseract_support/meshes/easo1.0/convex_decomposition/robot_base_decomposition_meshes/untitled_home_febert_Desktop_arm_base000_home_febert_Desktop_arm_base053.stl" /></geometry></collision>
+    <collision><geometry><mesh filename="package://tesseract_support/meshes/easo1.0/convex_decomposition/robot_base_decomposition_meshes/untitled_home_febert_Desktop_arm_base000_home_febert_Desktop_arm_base062.stl" /></geometry></collision>
+    <collision><geometry><mesh filename="package://tesseract_support/meshes/easo1.0/convex_decomposition/robot_base_decomposition_meshes/untitled_home_febert_Desktop_arm_base000_home_febert_Desktop_arm_base037.stl" /></geometry></collision>
+    <collision><geometry><mesh filename="package://tesseract_support/meshes/easo1.0/convex_decomposition/robot_base_decomposition_meshes/untitled_home_febert_Desktop_arm_base000_home_febert_Desktop_arm_base036.stl" /></geometry></collision>
+    <collision><geometry><mesh filename="package://tesseract_support/meshes/easo1.0/convex_decomposition/robot_base_decomposition_meshes/untitled_home_febert_Desktop_arm_base000_home_febert_Desktop_arm_base029.stl" /></geometry></collision>
+    <collision><geometry><mesh filename="package://tesseract_support/meshes/easo1.0/convex_decomposition/robot_base_decomposition_meshes/untitled_home_febert_Desktop_arm_base000_home_febert_Desktop_arm_base042.stl" /></geometry></collision>
+    <collision><geometry><mesh filename="package://tesseract_support/meshes/easo1.0/convex_decomposition/robot_base_decomposition_meshes/untitled_home_febert_Desktop_arm_base000_home_febert_Desktop_arm_base015.stl" /></geometry></collision>
+    <collision><geometry><mesh filename="package://tesseract_support/meshes/easo1.0/convex_decomposition/robot_base_decomposition_meshes/untitled_home_febert_Desktop_arm_base000_home_febert_Desktop_arm_base060.stl" /></geometry></collision>
+    <collision><geometry><mesh filename="package://tesseract_support/meshes/easo1.0/convex_decomposition/robot_base_decomposition_meshes/untitled_home_febert_Desktop_arm_base000_home_febert_Desktop_arm_base032.stl" /></geometry></collision>
+    <collision><geometry><mesh filename="package://tesseract_support/meshes/easo1.0/convex_decomposition/robot_base_decomposition_meshes/untitled_home_febert_Desktop_arm_base000_home_febert_Desktop_arm_base049.stl" /></geometry></collision>
+    <visual>
+      <origin xyz="0.55 0.5 0" rpy="0 0 0" />
+      <geometry>
+        <box size="0.1 2 2" />
+      </geometry>
+      <material name="Cyan">
+        <color rgba="0 1.0 1.0 1.0"/>
+      </material>
+    </visual>
     <collision>
+      <origin xyz="0.55 0.5 0" rpy="0 0 0" />
       <geometry>
-        <mesh filename="/home/febert/Desktop/arm_assembly_uniguide.STL"/>
+        <box size="0.1 2 2" />
       </geometry>
-      <material name="light_gray"/>
+      <material name="Cyan">
+        <color rgba="0 1.0 1.0 1.0"/>
+      </material>
     </collision>
-    <visual>
+    <!-- <visual>
       <origin xyz="0.55 0.0 0.43" rpy="0 0 0" />
      <geometry>
@@ -35,5 +74,5 @@
         <color rgba="0 1.0 1.0 1.0"/>
      </material>
-   </collision>
+   </collision> -->
   </link>
   <joint name="robot_base_joint" type ="fixed">

File: tesseract_support/urdf/easo1.0_whole.urdf (robot description, URDF)
Before this commit: robot easo1.0, 13 links, 12 joints
Links:
- link robot_base: geometry collision box size=0.1 2 2; collision mesh filename=package://tesseract_support/meshes/easo1.0/convex_decomposi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

Commit message: added endeff

File: tesseract_support/urdf/easo1.0_base_macro.xacro (robot description, xacro)
@@ -40,5 +40,5 @@
     <collision><geometry><mesh filename="package://tesseract_support/meshes/easo1.0/convex_decomposition/robot_base_decomposition_meshes/untitled_home_febert_Desktop_arm_base000_home_febert_Desktop_arm_base049.stl" /></geometry></collision>
     <visual>
-      <origin xyz="0.55 0.5 0" rpy="0 0 0" />
+      <origin xyz="0.9 0.5 0" rpy="0 0 0" />
       <geometry>
         <box size="0.1 2 2" />
@@ -49,5 +49,5 @@
     </visual>
     <collision>
-      <origin xyz="0.55 0.5 0" rpy="0 0 0" />
+      <origin xyz="0.9 0.5 0" rpy="0 0 0" />
       <geometry>
         <box size="0.1 2 2" />

File: tesseract_support/urdf/easo1.0_whole.urdf (robot description, URDF)
Before this commit: robot easo1.0, 13 links, 12 joints
Links:
- link arm_link7: geometry collision box size=0.14 0.16 0.1; collision cylinder length=0.289 radius=0.02
- link robot_base: geometry collision box size=0.1 2 2; collision mesh filename=package://tesseract_support/meshes/easo1.0/convex_decomposi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
Joints:
- joint joint_eef: origin xyz=0 0 0 rpy=0 0 0 -> xyz=-0.0525 0.029 0.289 rpy=0 0 0
- joint robot_base_joint: origin xyz=0.0 0.0 0.77153 rpy=0 0 0 -> xyz=0.0 0.0 0.0 rpy=0 0 0

File: tesseract_support/urdf/easo1.0_whole.xacro (robot description, xacro)
@@ -10,5 +10,5 @@
     <xacro:include filename="$(find tesseract_support)/urdf/easo1.0_base_macro.xacro"/>
     <xacro:workcell parent_link="world" >
-        <origin xyz="0.0 0.0 0.77153" rpy="0 0 0"/>
+        <origin xyz="0.0 0.0 0.0" rpy="0 0 0"/>
     </xacro:workcell >
     <joint name="robot_base_to_base_link" type="fixed">

File: tesseract_support/urdf/xarm7_macro.xacro (robot description, xacro)
@@ -222,4 +222,39 @@
         <origin rpy="0 0 0" xyz="0 0 0"/>
       </collision>
+      <visual>
+        <geometry>
+          <mesh filename="package://tesseract_support/meshes/easo1.0/visual/endeff_finger2_extd.stl"/>
+        </geometry>
+        <origin rpy="1.570796 0 0" xyz="0 0 0"/>
+        <material name="Silver"/>
+      </visual>
+      <visual>
+        <origin xyz="-0.0525 0.029 0.1445 " rpy="0 0 0"/>
+        <geometry>
+          <cylinder radius="0.01" length="0.289"/>
+        </geometry>
+        <material name="Silver"/>
+      </visual>
+      <collision>
+        <origin xyz="-0.0525 0.029 0.1445 " rpy="0 0 0"/>
+        <geometry>
+          <cylinder radius="0.02" length="0.289"/>
+        </geometry>
+        <material name="Silver"/>
+      </collision>
+      <visual>
+        <origin xyz="0.0 0 0.14" rpy="0 0 0" />
+        <geometry>
+          <box size="0.14 0.16 0.1" />
+        </geometry>
+        <material name="Silver"/>
+      </visual>
+      <collision>
+        <origin xyz="0.0 0 0.14" rpy="0 0 0" />
+        <geometry>
+          <box size="0.14 0.16 0.1" />
+        </geometry>
+        <material name="Silver"/>
+      </collision>
     </link>
     <joint name="joint7" type="revolute">
@@ -331,7 +366,8 @@
       <selfCollide>true</selfCollide>
     </gazebo>
-    <link name="tool0"/>
+    <link name="tool0">
+    </link>
     <joint name="joint_eef" type="fixed">
-      <origin rpy="0 0 0" xyz="0 0 0"/>
+      <origin rpy="0 0 0" xyz="-0.0525 0.029 0.289"/>
       <parent link="${prefix}link7"/>
       <child link="tool0"/>

Commit message: small changes to geometry

File: tesseract_support/urdf/easo1.0_base_macro.xacro (robot description, xacro)
@@ -40,5 +40,5 @@
     <collision><geometry><mesh filename="package://tesseract_support/meshes/easo1.0/convex_decomposition/robot_base_decomposition_meshes/untitled_home_febert_Desktop_arm_base000_home_febert_Desktop_arm_base049.stl" /></geometry></collision>
     <visual>
-      <origin xyz="0.9 0.5 0" rpy="0 0 0" />
+      <origin xyz="0.6 0.5 0" rpy="0 0 0" />
       <geometry>
         <box size="0.1 2 2" />
@@ -49,5 +49,5 @@
     </visual>
     <collision>
-      <origin xyz="0.9 0.5 0" rpy="0 0 0" />
+      <origin xyz="0.6 0.5 0" rpy="0 0 0" />
       <geometry>
         <box size="0.1 2 2" />

File: tesseract_support/urdf/easo1.0_whole.urdf (robot description, URDF)
Before this commit: robot easo1.0, 13 links, 12 joints
Links:
- link arm_link7: geometry collision box size=0.2 0.18 0.1; collision cylinder length=0.289 radius=0.02
- link robot_base: geometry collision box size=0.1 2 2; collision mesh filename=package://tesseract_support/meshes/easo1.0/convex_decomposi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

File: tesseract_support/urdf/xarm7_macro.xacro (robot description, xacro)
@@ -246,5 +246,5 @@
         <origin xyz="0.0 0 0.14" rpy="0 0 0" />
         <geometry>
-          <box size="0.14 0.16 0.1" />
+          <box size="0.2 0.18 0.1" />
         </geometry>
         <material name="Silver"/>
@@ -253,5 +253,5 @@
         <origin xyz="0.0 0 0.14" rpy="0 0 0" />
         <geometry>
-          <box size="0.14 0.16 0.1" />
+          <box size="0.2 0.18 0.1" />
         </geometry>
         <material name="Silver"/>
